File: PCB/WeatherStation/WeatherStation.kicad_pcb (KiCad board)
At the start: 2 copper layers, 31 parts, among them J1 LiPo, J2 Solar Panel, U1 TPS259621DDAT, U2 MIC5528-3.3YMT-TR, U3 ESP32-C3-MINI-1-N4, U4 BQ24040DSQR

Commit message: Rough draft of Control PCB with Gerbers
Parts:
- removed D1: Blue, LED_SMD:LED_0603_1608Metric_Pad1.05x0.95mm_HandSolder
- removed D2: Green, LED_SMD:LED_0603_1608Metric_Pad1.05x0.95mm_HandSolder
- removed D3: Red, LED_SMD:LED_0603_1608Metric_Pad1.05x0.95mm_HandSolder
- removed J1: LiPo, TerminalBlock:TerminalBlock_Altech_AK300-2_P5.00mm
- removed J2: Solar Panel, TerminalBlock:TerminalBlock_Altech_AK300-2_P5.00mm
- added Air1: Air Quality Sensor, Connector_PinHeader_2.54mm:PinHeader_1x03_P2.54mm_Vertical, F.Cu at (171.5, 129.8)
- added Bat1: LiPo, TerminalBlock:TerminalBlock_Altech_AK300-2_P5.00mm, F.Cu at (169.3, 85.0)
- added C10: 0.1u, Capacitor_SMD:C_0603_1608Metric_Pad1.08x0.95mm_HandSolder, F.Cu at (136.2, 131.0)
- added C11: 0.1u, Capacitor_SMD:C_0603_1608Metric_Pad1.08x0.95mm_HandSolder, F.Cu at (179.2, 103.8)
- added C12: 0.1u, Capacitor_SMD:C_0603_1608Metric_Pad1.08x0.95mm_HandSolder, F.Cu at (179.5, 116.8)
- added C13: 100u, Capacitor_THT:C_Radial_D5.0mm_H11.0mm_P2.00mm, F.Cu at (151.5, 91.8)
- added C14: 100u, Capacitor_THT:C_Radial_D6.3mm_H11.0mm_P2.50mm, F.Cu at (151.2, 100.0)
- added C15: 47u, Capacitor_THT:C_Radial_D4.0mm_H7.0mm_P1.50mm, F.Cu at (142.5, 120.5)
- added C16: 360p, Capacitor_SMD:C_0402_1005Metric_Pad0.74x0.62mm_HandSolder, F.Cu at (134.2, 101.0)
- added C17: 200p, Capacitor_SMD:C_0603_1608Metric_Pad1.08x0.95mm_HandSolder, F.Cu at (133.0, 127.1)
- added C18: 100u, Capacitor_THT:C_Radial_D5.0mm_H11.0mm_P2.00mm, F.Cu at (142.2, 113.2)
- added C9: 220u, Capacitor_THT:C_Radial_D5.0mm_H11.0mm_P2.00mm, F.Cu at (168.8, 96.5)
- added Charging1: G/Charging, LED_SMD:LED_0603_1608Metric_Pad1.05x0.95mm_HandSolder, F.Cu at (175.0, 98.2)
- added D6: S14, Diode_SMD:D_SOD-123F, F.Cu at (143.2, 103.8)
- added D7: S14, Diode_SMD:D_SOD-123F, F.Cu at (135.1, 121.5)
- added First1: B/First Charge, LED_SMD:LED_0603_1608Metric_Pad1.05x0.95mm_HandSolder, F.Cu at (188.0, 95.8)
- added JTAG1: JTAG, Connector_PinHeader_2.54mm:PinHeader_1x04_P2.54mm_Vertical, F.Cu at (163.9, 134.2)
- added L1: 100u, Inductor_THT:L_Toroid_Vertical_L10.2mm_W3.8mm_P3.8mm, F.Cu at (138.8, 88.2)
- added L2: 100u, Inductor_THT:L_Toroid_Vertical_L10.2mm_W3.8mm_P3.8mm, F.Cu at (137.8, 113.2)
- added Main1: G/Main, LED_SMD:LED_0603_1608Metric_Pad1.05x0.95mm_HandSolder, F.Cu at (155.2, 125.2)
- added Program1: Boot Mode, Button_Switch_THT:SW_PUSH_6mm_H5mm, F.Cu at (188.5, 107.5)
- added Q1: C1815, Package_TO_SOT_THT:TO-92, F.Cu at (147.7, 117.1)
- added Q2: 2N2222, Package_TO_SOT_THT:TO-92, F.Cu at (147.7, 124.1)
- added Q3: P2N2907A, Package_TO_SOT_THT:TO-92, F.Cu at (148.0, 110.1)
- added R16: 10k, Resistor_SMD:R_0603_1608Metric_Pad0.98x0.95mm_HandSolder, F.Cu at (159.5, 125.2)
- added R17: 402k, Resistor_SMD:R_0603_1608Metric_Pad0.98x0.95mm_HandSolder, F.Cu at (169.6, 106.8)
- added R18: 665k, Resistor_SMD:R_0603_1608Metric_Pad0.98x0.95mm_HandSolder, F.Cu at (173.6, 103.8)
- added R19: 1k, Resistor_SMD:R_0603_1608Metric_Pad0.98x0.95mm_HandSolder, F.Cu at (155.4, 122.2)
- added R20: 2.4M, Resistor_SMD:R_0603_1608Metric_Pad0.98x0.95mm_HandSolder, F.Cu at (173.6, 106.8)
- added R21: 2.4M, Resistor_SMD:R_0603_1608Metric_Pad0.98x0.95mm_HandSolder, F.Cu at (173.0, 117.0)
- added R22: 10k, Resistor_SMD:R_0603_1608Metric_Pad0.98x0.95mm_HandSolder, F.Cu at (188.2, 113.2)
- added R23: 10k, Resistor_SMD:R_0603_1608Metric_Pad0.98x0.95mm_HandSolder, F.Cu at (188.2, 115.0)
- added R24: 10k, Resistor_SMD:R_0603_1608Metric_Pad0.98x0.95mm_HandSolder, F.Cu at (155.3, 116.5)
- added R25: 1k, Resistor_SMD:R_0603_1608Metric_Pad0.98x0.95mm_HandSolder, F.Cu at (155.2, 119.2)
- added R26: 220, Resistor_SMD:R_0603_1608Metric_Pad0.98x0.95mm_HandSolder, F.Cu at (155.3, 113.5)
- added R27: 10k, Resistor_SMD:R_0603_1608Metric_Pad0.98x0.95mm_HandSolder, F.Cu at (148.0, 104.8)
- added R28: 1k, Resistor_SMD:R_0603_1608Metric_Pad0.98x0.95mm_HandSolder, F.Cu at (155.2, 107.5)
- added R29: 10k, Resistor_SMD:R_0603_1608Metric_Pad0.98x0.95mm_HandSolder, F.Cu at (142.5, 101.0)
- added R30: 1.18k, Resistor_SMD:R_0603_1608Metric_Pad0.98x0.95mm_HandSolder, F.Cu at (138.8, 104.2)
- added R31: 180, Resistor_SMD:R_0603_1608Metric_Pad0.98x0.95mm_HandSolder, F.Cu at (142.5, 97.8)
- added R32: 390m, Resistor_SMD:R_1206_3216Metric_Pad1.30x1.75mm_HandSolder, F.Cu at (146.8, 99.2)
- added R33: 10k, Resistor_SMD:R_0603_1608Metric_Pad0.98x0.95mm_HandSolder, F.Cu at (145.0, 128.5)
- added R34: 3.3k, Resistor_SMD:R_0603_1608Metric_Pad0.98x0.95mm_HandSolder, F.Cu at (149.3, 128.5)
- added R35: 180, Resistor_SMD:R_0603_1608Metric_Pad0.98x0.95mm_HandSolder, F.Cu at (139.2, 122.8)
- added R36: 680m, Resistor_SMD:R_0603_1608Metric_Pad0.98x0.95mm_HandSolder, F.Cu at (143.2, 125.0)
- added Rain1: Rain Sensor, Connector_PinHeader_2.54mm:PinHeader_1x02_P2.54mm_Vertical, F.Cu at (170.0, 113.0)
- added Rst1: Reset, Button_Switch_THT:SW_PUSH_6mm_H5mm, F.Cu at (145.6, 135.7)
- added Short1: R/Short, LED_SMD:LED_0603_1608Metric_Pad1.05x0.95mm_HandSolder, F.Cu at (169.8, 100.5)
- added SolarIn1: Solar Panel, TerminalBlock:TerminalBlock_Altech_AK300-2_P5.00mm, F.Cu at (182.4, 85.0)
- added U5: BME280, Imported:PSON65P250X250X100-8N, F.Cu at (182.2, 117.5)
- added U6: MC33063ADRJR, Imported:SON80P400X400X80-9N, F.Cu at (137.8, 99.8)
- added U7: MC33063ADRJR, Imported:SON80P400X400X80-9N, F.Cu at (137.4, 126.8)
- added U8: 74LVCH1T45GW, Package_TO_SOT_SMD:SOT-363_SC-70-6_Handsoldering, F.Cu at (162.0, 129.0)
- added UART1: UART, Connector_PinHeader_2.54mm:PinHeader_1x04_P2.54mm_Vertical, F.Cu at (150.5, 134.2)
- added UV1: UV Sensor, Connector_PinHeader_2.54mm:PinHeader_1x03_P2.54mm_Vertical, F.Cu at (182.8, 112.3)
- added Ultra1: Ultrasonic Sensor, Connector_PinHeader_2.54mm:PinHeader_1x04_P2.54mm_Vertical, F.Cu at (171.5, 122.8)
- added Wind1: B/Wind, LED_SMD:LED_0603_1608Metric_Pad1.05x0.95mm_HandSolder, F.Cu at (155.2, 110.5)
- added Wind_Sen1: Wind Sensor, Connector_PinHeader_2.54mm:PinHeader_1x03_P2.54mm_Vertical, F.Cu at (165.0, 113.0)
- R1: value 10k -> 665k
- R13: value 2k -> 1k
- R3: value 10k -> 220
- R9: value 10k -> 1k
- U3: value ESP32-C3-MINI-1-N4 -> ESP32-S2-MINI-1; footprint Imported:XCVR_ESP32-C3-MINI-1-N4 -> Imported:XCVR_ESP32-S2-MINI-1
- moved U3 77.8 mm to (182.3, 128.0), turned to -90 degrees
- moved C2 68.6 mm to (188.2, 117.0), turned to 180 degrees
- moved U4 66.4 mm to (183.0, 95.0), turned to 90 degrees
- moved C3 61.9 mm to (188.5, 119.0), turned to 180 degrees
- moved C1 55.7 mm to (133.2, 131.0), turned to -90 degrees
- moved R2 54.1 mm to (153.8, 130.0)
- moved C8 50.0 mm to (177.2, 108.8)
- moved R9 48.3 mm to (188.2, 111.5)
- moved R3 45.0 mm to (159.5, 122.2)
- moved U1 44.3 mm to (161.9, 101.2), turned to 90 degrees
- moved R5 40.7 mm to (184.5, 99.2), turned to 90 degrees
- moved R4 40.4 mm to (178.5, 99.2), turned to 90 degrees
- moved R8 40.1 mm to (181.5, 99.2), turned to 90 degrees
- moved R7 38.7 mm to (188.0, 99.0), turned to 180 degrees
- moved R6 36.3 mm to (188.0, 93.0), turned to 180 degrees
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Connections:
- C8 pad 1: Net-(C8-Pad1) -> VDD3.3
- C8 pad 2: Net-(C8-Pad2) -> GND
- R1 pad 1: VDD3.3 -> Net-(C4-Pad2)
- R1 pad 2: Net-(R1-Pad2) -> Solar
- R3 pad 1: Net-(R3-Pad1) -> Net-(Q2-Pad2)
- R3 pad 2: VDD3.3 -> Main Control
- R9 pad 1: Net-(R9-Pad1) -> Net-(C11-Pad1)
- R9 pad 2: unconnected-(R9-Pad2) -> Net-(R9-Pad2)
- U1 pad 5: unconnected-(U1-Pad5) -> VDDraw
- U2 pad 1: Net-(C8-Pad1) -> VDD3.3
- U2 pad 2: Net-(C8-Pad1) -> VDD3.3
- U2 pad 3: Net-(C8-Pad2) -> GND
- U2 pad 4: unconnected-(U2-Pad4) -> VDDraw
- U2 pad 6: unconnected-(U2-Pad6) -> VDDraw
- U2 pad 7: Net-(C8-Pad2) -> GND
- U3 pad 1: Net-(U3-Pad1) -> GND
- U3 pad 10: unconnected-(U3-Pad10) -> UV Power
- U3 pad 11: Net-(U3-Pad1) -> Solar
- U3 pad 12: unconnected-(U3-Pad12) -> Rain
- U3 pad 13: unconnected-(U3-Pad13) -> Rain Power
- U3 pad 14: Net-(U3-Pad1) -> Wind
- U3 pad 15: unconnected-(U3-Pad15) -> Wind Control
- U3 pad 16: unconnected-(U3-Pad16) -> Main Control
- U3 pad 17: unconnected-(U3-Pad17) -> Trig
- U3 pad 18: unconnected-(U3-Pad18) -> Echo
- U3 pad 2: Net-(U3-Pad1) -> GND
- U3 pad 21: unconnected-(U3-Pad21) -> PPM RX
- U3 pad 22: Net-(R3-Pad1) -> PPM TX
- U3 pad 23: Net-(R9-Pad1) -> unconnected-(U3-Pad23)
- U3 pad 30: unconnected-(U3-Pad30) -> GND
- U3 pad 35: unconnected-(U3-Pad35) -> /TCK
- U3 pad 36: Net-(U3-Pad1) -> /TDO
- U3 pad 37: Net-(U3-Pad1) -> /TDI
- U3 pad 38: Net-(U3-Pad1) -> /TMS
- U3 pad 39: Net-(U3-Pad1) -> /RX
- U3 pad 4: unconnected-(U3-Pad4) -> Net-(R9-Pad2)
- U3 pad 40: Net-(U3-Pad1) -> /TX
- U3 pad 41: Net-(U3-Pad1) -> unconnected-(U3-Pad41)
- U3 pad 42: Net-(U3-Pad1) -> GND
- U3 pad 43: Net-(U3-Pad1) -> GND
- U3 pad 44: Net-(U3-Pad1) -> unconnected-(U3-Pad44)
- U3 pad 45: Net-(U3-Pad1) -> Net-(C1-Pad2)
- U3 pad 46: Net-(U3-Pad1) -> GND
- U3 pad 47: Net-(U3-Pad1) -> GND
- U3 pad 48: Net-(U3-Pad1) -> GND
- U3 pad 5: Net-(R1-Pad2) -> Battery
- U3 pad 50: Net-(U3-Pad1) -> GND
- U3 pad 51: Net-(U3-Pad1) -> GND
- U3 pad 52: Net-(U3-Pad1) -> GND
- U3 pad 53: Net-(U3-Pad1) -> GND
- U3 pad 6: unconnected-(U3-Pad6) -> SCL
- U3 pad 7: unconnected-(U3-Pad7) -> SDA
- U3 pad 8: Net-(C1-Pad2) -> BME Power
- U3 pad 9: unconnected-(U3-Pad9) -> UV
Routing:
- net GND: track 0.00 -> 93.1 mm, vias 0 -> 32
- net VDDraw: track 0.00 -> 72.2 mm, vias 0 -> 3
- net Net-(C1-Pad2): track 0.00 -> 68.4 mm, vias 0 -> 1
- net Main Gnd: track 0.00 -> 58.4 mm, vias 0 -> 1
- net Main 5V: track 0.00 -> 36.0 mm, vias 0 -> 3
- net /TX: track 0.00 -> 32.9 mm, vias 0 -> 1
- net /RX: track 0.00 -> 30.0 mm
- net Wind Pow: track 0.00 -> 28.2 mm, vias 0 -> 1
- net Net-(C4-Pad2): track 0.00 -> 28.1 mm
- net Battery: track 0.00 -> 26.8 mm, vias 0 -> 2
- net Net-(D6-Pad2): track 0.00 -> 23.0 mm
- net Net-(L2-Pad1): track 0.00 -> 23.0 mm
- net Solar: track 0.00 -> 22.1 mm
- net Wind Control: track 0.00 -> 21.2 mm
- net BME Power: track 0.00 -> 20.7 mm, vias 0 -> 2
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- added copper zone on In1.Cu, net GND
- added copper zone on In2.Cu, net Main 5V
- added copper zone on In2.Cu, net Main Gnd
- added copper zone on In2.Cu, net VDD3.3
- added copper zone on In2.Cu, net Vbat
- added copper zone on In2.Cu, net Wind 12V
- added copper zone on In2.Cu, net Wind Pow
Other:
- board outline added: 60 x 60 mm
- copper layers 2 -> 4
- board text added: "12V"
- board text added: "3.3V"
- board text added: "5V"
- board text added: "Echo"
- board text added: "GND"
- board text added: "Logan Stranc Utah Valley University Weather Station v1.0"
- board text added: "Out"
- board text added: "RX"
- board text added: "TCK"
- board text added: "TDI"
- board text added: "TDO"
- board text added: "TMS"
- board text added: "TX"
- board text added: "Trig"
