File: PCB/WeatherStation/WeatherStation.kicad_sch (KiCad schematic)
At the start: 31 parts, among them J1 LiPo, J2 Solar Panel, U1 TPS259621DDAT, U2 MIC5528-3.3YMT-TR, U3 ESP32-C3-MINI-1-N4, U4 BQ24040DSQR

Commit message: Rough draft of Control PCB with Gerbers
Parts:
- removed U3: ESP32-C3-MINI-1-N4, XCVR_ESP32-C3-MINI-1-N4, symbol ESP32-C3-MINI-1-N4:ESP32-C3-MINI-1-N4
- added Air1: Air Quality Sensor, Connector_PinHeader_2.54mm:PinHeader_1x03_P2.54mm_Vertical, symbol Connector:Conn_01x03_Male
- added C10, C11, C12: 0.1u, Capacitor_SMD:C_0603_1608Metric_Pad1.08x0.95mm_HandSolder, symbol Device:C
- added C13, C18: 100u, Capacitor_THT:C_Radial_D5.0mm_H11.0mm_P2.00mm, symbol Device:C_Polarized
- added C14: 100u, Capacitor_THT:C_Radial_D6.3mm_H11.0mm_P2.50mm, symbol Device:C_Polarized
- added C15: 47u, Capacitor_THT:C_Radial_D4.0mm_H7.0mm_P1.50mm, symbol Device:C_Polarized
- added C16: 360p, Capacitor_SMD:C_0402_1005Metric_Pad0.74x0.62mm_HandSolder, symbol Device:C
- added C17: 200p, Capacitor_SMD:C_0603_1608Metric_Pad1.08x0.95mm_HandSolder, symbol Device:C
- added C9: 220u, Capacitor_THT:C_Radial_D5.0mm_H11.0mm_P2.00mm, symbol Device:C_Polarized
- added D6, D7: S14, Diode_SMD:D_SOD-123F, symbol Device:D_Schottky
- added JTAG1: JTAG, Connector_PinHeader_2.54mm:PinHeader_1x04_P2.54mm_Vertical, symbol Connector:Conn_01x04_Male
- added L1, L2: 100u, Inductor_THT:L_Toroid_Vertical_L10.2mm_W3.8mm_P3.8mm, symbol Device:L_Ferrite
- added Main1: G/Main, LED_SMD:LED_0603_1608Metric_Pad1.05x0.95mm_HandSolder, symbol Device:LED
- added Program1: Boot Mode, Button_Switch_THT:SW_PUSH_6mm_H5mm, symbol Switch:SW_SPST
- added Q1: C1815, Package_TO_SOT_THT:TO-92, symbol Device:Q_NPN_ECB
- added Q2: 2N2222, Package_TO_SOT_THT:TO-92, symbol Device:Q_NPN_CBE
- added Q3: P2N2907A, Package_TO_SOT_THT:TO-92, symbol Device:Q_PNP_CBE
- added R16, R22, R23, R24, R27, R29, R33: 10k, Resistor_SMD:R_0603_1608Metric_Pad0.98x0.95mm_HandSolder, symbol Device:R_Small_US
- added R17: 402k, Resistor_SMD:R_0603_1608Metric_Pad0.98x0.95mm_HandSolder, symbol Device:R_Small_US
- added R18: 665k, Resistor_SMD:R_0603_1608Metric_Pad0.98x0.95mm_HandSolder, symbol Device:R_Small_US
- added R19, R25, R28: 1k, Resistor_SMD:R_0603_1608Metric_Pad0.98x0.95mm_HandSolder, symbol Device:R_Small_US
- added R20, R21: 2.4M, Resistor_SMD:R_0603_1608Metric_Pad0.98x0.95mm_HandSolder, symbol Device:R_Small_US
- added R26: 220, Resistor_SMD:R_0603_1608Metric_Pad0.98x0.95mm_HandSolder, symbol Device:R_Small_US
- added R30: 1.18k, Resistor_SMD:R_0603_1608Metric_Pad0.98x0.95mm_HandSolder, symbol Device:R_Small_US
- added R31, R35: 180, Resistor_SMD:R_0603_1608Metric_Pad0.98x0.95mm_HandSolder, symbol Device:R_Small_US
- added R32: 390m, Resistor_SMD:R_1206_3216Metric_Pad1.30x1.75mm_HandSolder, symbol Device:R_Small_US
- added R34: 3.3k, Resistor_SMD:R_0603_1608Metric_Pad0.98x0.95mm_HandSolder, symbol Device:R_Small_US
- added R36: 680m, Resistor_SMD:R_0603_1608Metric_Pad0.98x0.95mm_HandSolder, symbol Device:R_Small_US
- added Rain1: Rain Sensor, Connector_PinHeader_2.54mm:PinHeader_1x02_P2.54mm_Vertical, symbol Connector:Conn_01x02_Male
- added Rst1: Reset, Button_Switch_THT:SW_PUSH_6mm_H5mm, symbol Switch:SW_SPST
- added U3: ESP32-S2-MINI-1, Imported:XCVR_ESP32-S2-MINI-1, symbol ESP32-S2-MINI-1:ESP32-S2-MINI-1
- added U5: BME280, Imported:PSON65P250X250X100-8N, symbol BME280:BME280
- added U6, U7: MC33063ADRJR, Imported:SON80P400X400X80-9N, symbol MC33063ADRJR:MC33063ADRJR
- added U8: 74LVCH1T45GW, Package_TO_SOT_SMD:SOT-363_SC-70-6_Handsoldering, symbol 74LVCH1T45GW:74LVCH1T45GW
- added UART1: UART, Connector_PinHeader_2.54mm:PinHeader_1x04_P2.54mm_Vertical, symbol Connector:Conn_01x04_Male
- added UV1: UV Sensor, Connector_PinHeader_2.54mm:PinHeader_1x03_P2.54mm_Vertical, symbol Connector:Conn_01x03_Male
- added Ultra1: Ultrasonic Sensor, Connector_PinHeader_2.54mm:PinHeader_1x04_P2.54mm_Vertical, symbol Connector:Conn_01x04_Male
- added Wind1: B/Wind, LED_SMD:LED_0603_1608Metric_Pad1.05x0.95mm_HandSolder, symbol Device:LED
- added Wind_Sen1: Wind Sensor, Connector_PinHeader_2.54mm:PinHeader_1x03_P2.54mm_Vertical, symbol Connector:Conn_01x03_Male
- Charging1: renamed from D2; value Green -> G/Charging
- First1: renamed from D1; value Blue -> B/First Charge
- R1: value 10k -> 665k
- R13: value 2k -> 1k
- R3: value 10k -> 220
- R9: value 10k -> 1k
- Short1: renamed from D3; value Red -> R/Short
- U1: footprint VREG_LM5017MR/NOPB -> Imported:VREG_LM5017MR_NOPB
- U2: footprint SON40P120X120X60-7N -> Imported:SON40P120X120X60-7N
- U4: footprint SON40P200X200X80-11N -> Imported:SON40P200X200X80-11N
- renumbered J1 to Bat1, J2 to SolarIn1
Connections:
- net GND: now also C8.2, U2.3 (GND), U2.7 (GND), C10.2, C11.2, C12.2, C13.2, C14.2, C16.2, C9.2, Program1.2 (B), Q1.1 (E), Q2.3 (E), R16.1, R17.2, R20.2, R24.2, R28.2, R30.1, Rain1.2 (Pin_2), Rst1.2 (B), U3.1 (GND), U3.2 (GND), U3.30 (GND), U3.42 (GND), U3.43 (GND), U3.46 (GND), U3.47 (GND), U3.48 (GND), U3.49 (GND), U3.50 (GND), U3.51 (GND), U3.52 (GND), U3.53 (GND), U3.54 (GND), U3.55 (GND), U3.56 (GND), U3.57 (GND), U3.58 (GND), U3.59 (GND), U3.60 (GND), U3.61 (GND), U3.61_1 (GND), U3.61_2 (GND), U3.61_3 (GND), U3.61_4 (GND), U3.61_5 (GND), U3.61_6 (GND), U3.61_7 (GND), U3.61_8 (GND), U3.62 (GND), U3.63 (GND), U3.64 (GND), U3.65 (GND), U5.1 (GND), U5.5 (SDO), U5.7 (GND), U6.2 (SWITCH_EMITTER), U6.4 (GND), U6.9 (EXP), UART1.1 (Pin_1), UV1.2 (Pin_2), Wind_Sen1.3 (Pin_3)
- net VDD3.3: now also C8.1, U2.1 (VOUT), U2.2 (VOUT), Main1.2 (A), U3.3 (3V3), U8.1 (VCC(A)), UART1.4 (Pin_4); no longer R1.1, R3.2
- net Vbat: now also R18.1
- net VDDraw: now reaches U2.4 (EN)
- net VDDraw: now also U1.5 (OUT), U2.6 (VIN), C18.1, C9.1, Q3.1 (C), R27.1, R36.2, U7.6 (VCC)
- net at C4.2, SolarIn1.2 (Pin_2), U4.1 (IN): now also R1.1
- net at C1.2, R2.1: now also C10.1, Rst1.1 (A), U3.45 (EN)
- net at R3.1: now also Q2.2 (B), R16.2
- net at R9.1: now also C11.1, Program1.1 (A)
- net Solar: now reaches R1.2
- net Solar: now also R17.1, U3.11 (IO7)
- net at R9.2: now also U3.4 (IO0)
- new net: L2.1, R35.1, R36.1, U7.7 (IPK)
- new net: D7.2 (A), L2.2, U7.1 (SWITCH_COLLECTOR)
- new net: Q1.2 (C), R26.1
- new net: Q3.2 (B), R26.2, R27.2
- new net: R33.1, R34.1, U7.5 (COMPARATOR_INVERTING_INPUT)
- new net: L1.1, R31.1, R32.1, U6.7 (IPK)
- new net: D6.2 (A), L1.2, U6.1 (SWITCH_COLLECTOR)
- new net: C16.1, U6.3 (TIMING_CAPACITOR)
- new net: C17.1, U7.3 (TIMING_CAPACITOR)
- new net: R35.2, U7.8 (DRIVER_COLLECTOR)
- new net: Main1.1 (K), R19.1
- new net: Q1.3 (B), R24.1, R25.2
- new net: R29.1, R30.2, U6.5 (COMPARATOR_INVERTING_INPUT)
- new net: R31.2, U6.8 (DRIVER_COLLECTOR)
- new net: R28.1, Wind1.1 (K)
- new net BME Power: C12.1, R22.1, R23.1, U3.8 (IO4), U5.2 (CSB), U5.6 (VDDIO), U5.8 (VDD)
- new net Battery: R18.2, R20.1, U3.5 (IO1)
- new net Echo: U3.18 (IO14), U8.3 (A)
- new net Echo High: U8.4 (B), Ultra1.2 (Pin_2)
- new net Main 5V: Air1.2 (Pin_2), C15.1, D7.1 (K), R33.2, U8.6 (VCC(B)), Ultra1.4 (Pin_4)
- new net Main Control: R3.2, U3.16 (IO12)
- new net Main Gnd: Air1.3 (Pin_3), C15.2, C17.2, C18.2, Q2.1 (C), R19.2, R34.2, U7.2 (SWITCH_EMITTER), U7.4 (GND), U7.9 (EXP), U8.2 (GND), U8.5 (DIR), Ultra1.3 (Pin_3)
- new net PPM RX: Air1.1 (Pin_1), U3.21 (IO17)
- new net PPM TX: U3.22 (IO18)
- new net RX: U3.39 (TXD0), UART1.3 (Pin_3)
- new net Rain: R21.1, Rain1.1 (Pin_1), U3.12 (IO8)
- new net Rain Power: R21.2, U3.13 (IO9)
- new net SCL: R23.2, U3.6 (IO2), U5.4 (SCK)
- new net SDA: R22.2, U3.7 (IO3), U5.3 (SDI)
- new net TCK: JTAG1.4 (Pin_4), U3.35 (IO39)
- new net TDI: JTAG1.2 (Pin_2), U3.37 (IO41)
- new net TDO: JTAG1.3 (Pin_3), U3.36 (IO40)
- new net TMS: JTAG1.1 (Pin_1), U3.38 (IO42)
- new net TX: U3.40 (RXD0), UART1.2 (Pin_2)
- new net Trig: U3.17 (IO13), Ultra1.1 (Pin_1)
- new net UV: U3.9 (IO5), UV1.1 (Pin_1)
- new net UV Power: U3.10 (IO6), UV1.3 (Pin_3)
- new net Wind: U3.14 (IO10), Wind_Sen1.1 (Pin_1)
- new net Wind 12V: C14.1, D6.1 (K), R29.2, Wind_Sen1.2 (Pin_2)
- new net Wind Control: R25.1, U3.15 (IO11)
- new net Wind Pow: C13.1, Q3.3 (E), R32.2, U6.6 (VCC), Wind1.2 (A)
- no-connect marks 0 -> 4
Other:
- note added: "3.28V max to analog in"
- note added: "Boost Converter 4.2V to for Ultrasonic Snow sensor and Air Quality sensor"
- note added: "Boost Converter 4.2V to for Wind sensor"
- note added: "Control Transistor for Air quality and Ultrasonic sensor"
- note added: "Control Transistor for Wind sensor"
- note added: "DIR to Gnd means B to A"
- note added: "DVDT estimated for moderate value. UVLO voltage divider means under-volate of 3.19V ILM of 1K means 0.91A output current limit OVSEL 402k to ground means over-voltage of 5.7V"
- note added: "Efuse for Lipo discharge safety."
- note added: "IO45 and IO46 are used for booting"
- note added: "ISet 1k sets charge current to 540mA max. ISet2 pulled low means ISet current is used Preterm floating sets finishing current to 10% and start current to 20%. TS disabled is pulled low."
- note added: "Lipo Charger from Solar"
- note added: "Logic Level Converter"
- note added: "Temperature, Humidity and Pressure sensor"
- note added: "Voltage Regulator 4.2V to 3.3V"
- moved on the sheet: C1, C2, C3, C4, C5, Charging1, First1, R2, R4, R5, R6, R7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
